Commit message: Add aruco marker to husky

File: husky_description/urdf/accessories/vlp16_mount.urdf.xacro (robot description, xacro)
@@ -7,10 +7,10 @@
     -->
     <link name="${prefix}vlp16_mount_base_link" />
-    <link name="${prefix}vlp16_mount_plate">
+    <link name="${prefix}vlp16_mount_left_support">
       <visual>
         <geometry>
-          <box size="0.04 0.141 0.0063" />
+          <box size="0.012 0.012 ${height}" />
         </geometry>
-        <material name="black">
+        <material name="white">
           <color rgba="1 1 1 1" />
         </material>
@@ -19,22 +19,5 @@
       <collision>
         <geometry>
-          <box size="0.04 0.02 ${height}" />
-        </geometry>
-        <origin xyz="0 0 0" rpy="0 0 0" />
-      </collision>
-    </link>
-    <link name="${prefix}vlp16_mount_left_support">
-      <visual>
-        <geometry>
-          <box size="0.04 0.02 ${height}" />
-        </geometry>
-        <material name="black">
-          <color rgba="1 1 1 1" />
-        </material>
-        <origin xyz="0 0 0" rpy="0 0 0" />
-      </visual>
-      <collision>
-        <geometry>
-          <box size="0.04 0.02 ${height}" />
+          <box size="0.012 0.012 ${height}" />
         </geometry>
         <origin xyz="0 0 0" rpy="0 0 0" />
@@ -44,7 +27,7 @@
       <visual>
         <geometry>
-          <box size="0.04 0.02 ${height}" />
+          <box size="0.012 0.012 ${height}" />
         </geometry>
-        <material name="black">
+        <material name="white">
           <color rgba="1 1 1 1" />
         </material>
@@ -53,5 +36,5 @@
       <collision>
         <geometry>
-          <box size="0.04 0.02 ${height}" />
+          <box size="0.012 0.012 ${height}" />
         </geometry>
         <origin xyz="0 0 0" rpy="0 0 0" />
@@ -66,18 +49,13 @@
       <parent link="${prefix}vlp16_mount_base_link" />
       <child link="${prefix}vlp16_mount_left_support" />
-      <origin xyz="0 0.06 ${height/2}" rpy="0 0 0"/>
+      <origin xyz="0 0.04 ${height/2}" rpy="0 0 0"/>
     </joint>
     <joint name="${prefix}vlp16_mount_right_support_joint" type="fixed">
       <parent link="${prefix}vlp16_mount_base_link" />
       <child link="${prefix}vlp16_mount_right_support" />
-      <origin xyz="0 -0.06 ${height/2}" rpy="0 0 0"/>
+      <origin xyz="0 -0.04 ${height/2}" rpy="0 0 0"/>
     </joint>
-    <joint name="${prefix}vlp16_mount_plate_joint" type="fixed">
-      <parent link="${prefix}vlp16_mount_base_link" />
-      <child link="${prefix}vlp16_mount_plate" />
-      <origin xyz="0 0 ${height}" rpy="0 0 0"/>
-    </joint>
-    <xacro:VLP-16 parent="${prefix}vlp16_mount_plate" topic="${topic}">
-      <origin xyz="0 0 0" rpy="0 0 0" />
+    <xacro:VLP-16 parent="${prefix}vlp16_mount_base_link" topic="${topic}">
+      <origin xyz="0 0 ${height}" rpy="0 0 0" />
     </xacro:VLP-16>
   </xacro:macro>

File: husky_description/urdf/decorations.urdf.xacro (robot description, xacro)
@@ -210,4 +210,54 @@
       <link name="top_plate_rear_link"/>
     </xacro:if>
+    <!-- connection link -->
+    <link name = "connection">
+      <visual>
+        <geometry>
+          <box size="0.1 0.1 1.0" />
+        </geometry>
+      </visual>
+      <collision>
+        <geometry>
+          <box size="0.1 0.1 0.3" />
+        </geometry>
+      </collision>
+      <inertial>
+            <mass value="2" />
+            <inertia ixx="0" ixy="0" ixz="0" iyy="0" iyz="0" izz="0" />
+        </inertial>
+    </link>
+    <gazebo reference="connection">
+    </gazebo>
+    <!-- Attach connection to top plate -->
+    <joint name="connection_joint" type="fixed">
+      <parent link="top_plate_link" />
+      <child link="connection" />
+      <origin xyz="0 0 0.5" rpy="0 0 0" />
+    </joint>
+    <!-- Aruco marker link -->
+    <link name = "Aruco_marker">
+      <visual>
+        <geometry>
+          <mesh filename="package://husky_description/meshes/Aruco_marker.dae" />
+        </geometry>
+      </visual>
+      <collision>
+        <geometry>
+          <mesh filename="package://husky_description/meshes/Aruco_marker.dae" />
+        </geometry>
+      </collision>
+      <inertial>
+            <mass value="4" />
+            <inertia ixx="0" ixy="0" ixz="0" iyy="0" iyz="0" izz="0" />
+        </inertial>
+    </link>
+    <gazebo reference="Aruco_marker">
+    </gazebo>
+    <!-- Attach Aruco_marker to connection -->
+    <joint name="Aruco_marker_joint" type="fixed">
+      <parent link="connection" />
+      <child link="Aruco_marker" />
+      <origin xyz="0 0 0.5" rpy="1.5707963 -1.5707963 0" />
+    </joint>
   </xacro:macro>
 </robot>

File: husky_description/urdf/husky.urdf.xacro (robot description, xacro)
@@ -59,7 +59,7 @@
   <xacro:include filename="$(find husky_description)/urdf/wheel.urdf.xacro" />
   <xacro:include filename="$(find husky_description)/urdf/accessories/intel_realsense.urdf.xacro"/>
-  <xacro:include filename="$(find husky_description)/urdf/accessories/hokuyo_ust10.urdf.xacro" />
   <xacro:include filename="$(find husky_description)/urdf/accessories/sick_lms1xx_mount.urdf.xacro"/>
   <xacro:include filename="$(find husky_description)/urdf/accessories/sensor_arch.urdf.xacro"/>
+  <xacro:include filename="$(find husky_description)/urdf/accessories/hokuyo_ust10.urdf.xacro"/>
   <xacro:include filename="$(find husky_description)/urdf/accessories/vlp16_mount.urdf.xacro"/>
   <xacro:property name="M_PI" value="3.14159"/>
